File: Board/Milled/Nyan.sch (EAGLE design)
At the start: 21 parts, among them IC1 74HCT541N, T1 TSM2314CX, U1 BLUEPILL455, U2 A4988_STEP, U3 MAX6966, X1 WR-WTB2.0-2_THT-VER, X2 WR-WTB2.0-4_THT_VER, X3 WR-WTB2.0-4_THT_VER, X4 WR-WTB2.0-5_THT-VER, X6 68610614122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

Commit message: Current development state with hardware fixes for 3 to 5 volt level shifting
Connections:
- removed net N$10: IC1A.Y1
- removed net N$11: IC1A.Y2
- removed net N$12: IC1A.Y3
- removed net N$13: IC1A.Y4
- removed net N$14: IC1A.Y5
- removed net N$15: IC1A.Y6
- removed net N$16: IC1A.Y7
- removed net N$17: IC1A.Y8
- removed net N$18: IC1A.A1
- removed net N$19: IC1A.A2
- removed net N$20: IC1A.A3
- removed net N$21: IC1A.A4
- removed net N$22: IC1A.A5
- removed net N$23: IC1A.A6
- removed net N$24: IC1A.A7
- removed net N$25: IC1A.A8
- removed net N$8: R3.1, T1.D
- removed net N$9: T1.G
- net D1: now also IC1A.A1
- net D1_5V: now also IC1A.Y1
- net D2: now also IC1A.A2
- net D2_5V: now also IC1A.Y2
- net D3: now also IC1A.A3
- net D3_5V: now also IC1A.Y3
- net D4: now also IC1A.A4
- net D4_5V: now also IC1A.Y4
- net D5: now also IC1A.A5
- net D5_5V: now also IC1A.Y5
- net D6: now also IC1A.A6
- net D6_5V: now also IC1A.Y6
- net DCLK: now also IC1A.A7
- net DCLK_5V: now also IC1A.Y7
- net LATCH: now also T1.G
- net LATCH_5V: now also R3.1, T1.D
- net STROBE: now also IC1A.A8
- net STROBE_5V: now also IC1A.Y8
